File: nrfmicro.kicad_pcb (KiCad board)
At the start: 2 copper layers, 18 x 33.3 mm, 26 parts, among them J1 USB_OTG, J2 USB_C_Receptacle_USB2.0, J3 Serial Connector, J4 Conn_01x02, Q1 DMG2305, SW1 SW_SPDT, U2 ProMicro, U3 AP2112K-3.3, U4 MCP73831-2-OT, U5 E73-2G4M08S1C-52840, Y2 32,768

Commit message: fixed solder mask clearance
Other:
- rule pad_to_mask_clearance: 0.2 -> 0
Changed lines of the file:
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@@
     (pad_size 3.25 3.25)
     (pad_drill 0)
-    (pad_to_mask_clearance 0.2)
-    (solder_mask_min_width 0.25)
+    (pad_to_mask_clearance 0)
     (aux_axis_origin 0 0)
     (grid_origin 96.181533 140.292775)
